File: memory.sch (KiCad schematic (older format))
At the start: 9 parts, among them U5 IS42S16400J-xC

Commit message: almost done with draft 1 of layout
Connections:
- net CLK: now reaches R34.1, U5.38 (CLK)
Changed lines of the file:
@@
 Wire Wire Line
 	8650 1700 8650 1850
+Text Label 4850 4050 0    50   ~ 0
+CLK
 $EndSCHEMATC
