File: Exodus1000.kicad_pcb (KiCad board)
At the start: 4 copper layers, 141.5 x 64.5 mm, 96 parts, among them J1 ARJ-169, J2 USB_B_Mini, J3 Conn_01x02, J4 Micro_SD_Card, M1 ET60S-02-24-02-X-VP-GP, M2 ET60S-02-24-02-X-VP-GP, M3 ET60S-02-24-02-X-VP-GP, M4 ET60S-02-24-02-X-VP-GP, U1 TM4C1294NCPDTGOOD, U2 93LCxxB, U3 FT232H, U4 tusb2077a, U5 IS42S16400J-xC, U6 74LS125, Y1 Crystal_GND24, Y2 Crystal_GND24, Y3 Crystal_GND24

Commit message: this is just a mess. but I think the schematic is basically right still.
Parts:
- removed C17, C18, C19, C20, C21, C22, C23, C24, C25, C26, C27, C28, C29, C30, C31, C32, C33, C34, C35, C36, C37, C38, C39: C_Small, Capacitor_SMD:C_0603_1608Metric
- removed J2: USB_B_Mini, Connector_USB:USB_Mini-B_Lumberg_2486_01_Horizontal
- removed J4: Micro_SD_Card, Connector_Card:microSD_HC_Wuerth_693072010801
- removed M1, M2, M3, M4: ET60S-02-24-02-X-VP-GP, Exodus_Connectors:ET60S-02-24-02-X-VP-GP
- removed R24, R25, R26, R27, R28, R29, R31, R32, R33, R35, R36, R37: R_Small, Resistor_SMD:R_0603_1608Metric
- removed R34: 0, Resistor_SMD:R_0603_1608Metric
- removed U5: IS42S16400J-xC, Package_SO:TSOP-II-54_22.2x10.16mm_P0.8mm
- removed U6: 74LS125, Package_SO:SOIC-14_3.9x8.7mm_P1.27mm
- removed Y3: Crystal_GND24, Crystal:Crystal_SMD_SeikoEpson_FA238-4Pin_3.2x2.5mm
- added 1: ET60S-02-24-02-X-VP-GP, Exodus_Connectors:ET60S-02-24-02-X-VP-GP, F.Cu at (58.4, 99.1)
- added 2: ET60S-02-24-02-X-VP-GP, Exodus_Connectors:ET60S-02-24-02-X-VP-GP, F.Cu at (91.4, 99.1)
- added 3: ET60S-02-24-02-X-VP-GP, Exodus_Connectors:ET60S-02-24-02-X-VP-GP, F.Cu at (124.5, 99.1)
- added 4: ET60S-02-24-02-X-VP-GP, Exodus_Connectors:ET60S-02-24-02-X-VP-GP, F.Cu at (78.7, 147.3)
- C1, C9: value 2.2u -> C_Small
- C11, C13, R3: moved to F.Cu
- C2, C6, C8: value 0.1u -> C_Small
- C3, C4: value 12p -> C_Small
- C5: value 1.0u -> C_Small
- J1: value ARJ-169 -> USB_B_Mini; footprint Exodus_Connectors:ARJ-169 -> Connector_USB:USB_Mini-B_Lumberg_2486_01_Horizontal
- R1: value 2k -> R_Small
- R2: value 4.87k 1% -> R_Small
- U1: value TM4C1294NCPDTGOOD -> 74LS125; footprint Package_QFP:TQFP-128_14x14mm_P0.4mm -> Package_SO:SOIC-14_3.9x8.7mm_P1.27mm
- U2: value 93LCxxB -> tusb2077a; footprint Package_SO:SOIC-8_3.9x4.9mm_P1.27mm -> Package_QFP:TQFP-48_7x7mm_P0.5mm; moved to F.Cu
- U3: value FT232H -> 93LCxxB; footprint Package_QFP:LQFP-48_7x7mm_P0.5mm -> Package_SO:SOIC-8_3.9x4.9mm_P1.27mm
- U4: value tusb2077a -> FT232H; footprint Package_QFP:TQFP-48_7x7mm_P0.5mm -> Package_QFP:LQFP-48_7x7mm_P0.5mm
- Y1: footprint Crystal:Crystal_SMD_3225-4Pin_3.2x2.5mm -> Crystal:Crystal_SMD_SeikoEpson_FA238-4Pin_3.2x2.5mm
- moved R16 59.0 mm to (200.7, 120.4)
- moved R15 54.0 mm to (187.7, 86.6)
- moved J3 50.3 mm to (150.5, 72.4)
- moved R17 49.0 mm to (202.2, 120.4), turned to 90 degrees
- moved R18 46.5 mm to (200.7, 117.4), turned to 90 degrees
- moved U2 42.9 mm to (147.3, 87.6), turned to 270 degrees
- moved J1 39.5 mm to (189.6, 115.9)
- moved R1 34.7 mm to (189.2, 87.8), turned to 90 degrees
- moved C13 31.3 mm to (138.4, 99.1), turned to 90 degrees
- moved C11 31.0 mm to (140.3, 99.2), turned to 90 degrees
- moved C4 30.6 mm to (186.2, 89.6), turned to 90 degrees
- moved C3 30.5 mm to (187.7, 92.6), turned to 90 degrees
- moved Y1 29.9 mm to (187.1, 96.2), turned to 90 degrees
- moved R2 29.5 mm to (190.7, 90.8)
- moved C5 25.9 mm to (191.1, 93.9), turned to 90 degrees
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Connections:
- net Net-(U4-Pad19) renamed /sheet5CBA03CB/ADBUS6
- net Net-(U4-Pad20) renamed /sheet5CBA03CB/ADBUS7
- net Net-(U4-Pad25) renamed /sheet5CBA03CB/ACBUS1
- net Net-(U4-Pad28) renamed /sheet5CBA03CB/ACBUS4
- net Net-(U4-Pad29) renamed /sheet5CBA03CB/ACBUS5
- net Net-(U4-Pad32) renamed /sheet5CBA03CB/ACBUS8
- net Net-(U4-Pad33) renamed /sheet5CBA03CB/ACBUS9
- C1 pad 1: +3V3 -> /D0_P
- C10 pad 1: +3V3 -> /sheet5CBA03CA/DM4
- C12 pad 1: /Connectors/sheet5C96EC1B/OSC1 -> /sheet5CBA03CB/OSC1
- C14 pad 1: /Connectors/sheet5C96EC1B/OSC0_R -> /sheet5CBA03CB/OSC0_R
- C2 pad 1: +3V3 -> /D0_N
- C3 pad 1: /TM4C129/OSC0 -> GND
- C3 pad 2: GND -> Net-(C3-Pad2)
- C5 pad 1: Net-(C5-Pad1) -> /sheet5CBA03CA/DP3
- C6 pad 1: +3V3 -> /sheet5CBA03CA/DM3
- C7 pad 1: Net-(C5-Pad1) -> /sheet5CBA03CA/DP1
- C8 pad 1: +3V3 -> /sheet5CBA03CA/DM1
- C9 pad 1: Net-(C5-Pad1) -> /sheet5CBA03CA/DP4
- R1 pad 1: /TM4C129/OSC1 -> /sheet5CBA03CA/DP0
- R1 pad 2: Net-(C4-Pad2) -> /D0_P
- R10 pad 1: /Connectors/D3_N -> GND
- R10 pad 2: /Connectors/sheet5C922FED/DM3 -> /D3_P
- R11 pad 1: /Connectors/D1_P -> GND
- R11 pad 2: /Connectors/sheet5C922FED/DP1 -> /D3_N
- R12 pad 1: /Connectors/D1_N -> GND
- R12 pad 2: /Connectors/sheet5C922FED/DM1 -> /D1_P
- R13 pad 1: /Connectors/D4_P -> GND
- R13 pad 2: /Connectors/sheet5C922FED/DP4 -> /D1_N
- R14 pad 1: /Connectors/D4_N -> GND
- R14 pad 2: /Connectors/sheet5C922FED/DM4 -> /D4_P
- R15 pad 1: /Connectors/D2_P -> GND
- R15 pad 2: /Connectors/sheet5C922FED/DP2 -> /D4_N
- R16 pad 1: /Connectors/D2_N -> Net-(R16-Pad1)
- R16 pad 2: /Connectors/sheet5C922FED/DM2 -> Net-(R16-Pad2)
- R17 pad 1: /Connectors/D5_P -> /sheet5CBA03CB/OSC0
- R17 pad 2: /Connectors/sheet5C922FED/DP5 -> /sheet5CBA03CB/OSC0_R
- R18 pad 1: /Connectors/D5_N -> Net-(R18-Pad1)
- R18 pad 2: /Connectors/sheet5C922FED/DM5 -> +3V3
- R19 pad 1: GND -> Net-(R19-Pad1)
- R19 pad 2: /Connectors/D3_P -> GND
- R2 pad 1: Net-(R2-Pad1) -> /sheet5CBA03CA/DM0
- R2 pad 2: GND -> /D0_N
- R20 pad 1: GND -> /BOARD_SENSE_4
- R20 pad 2: /Connectors/D3_N -> GND
- R21 pad 1: GND -> /BOARD_SENSE_3
- R21 pad 2: /Connectors/D1_P -> GND
- R22 pad 1: GND -> /BOARD_SENSE_1
- R22 pad 2: /Connectors/D1_N -> GND
- R23 pad 1: GND -> /BOARD_SENSE_2
- R23 pad 2: /Connectors/D4_P -> GND
- R3 pad 2: Net-(R3-Pad2) -> /sheet5CBA03CA/DP0
- R4 pad 1: /Connectors/sheet5C96EC1B/OSC0 -> /D3_P
- R4 pad 2: /Connectors/sheet5C96EC1B/OSC0_R -> /sheet5CBA03CA/DP3
- R5 pad 1: Net-(R5-Pad1) -> /D3_N
- R5 pad 2: +3V3 -> /sheet5CBA03CA/DM3
- R6 pad 1: /Connectors/sheet5C922FED/DP0 -> /D1_P
- R6 pad 2: /TM4C129/USB_D_P -> /sheet5CBA03CA/DP1
- R7 pad 1: /Connectors/sheet5C922FED/DM0 -> /D1_N
- R7 pad 2: /TM4C129/USB_D_N -> /sheet5CBA03CA/DM1
- R8 pad 1: Net-(R8-Pad1) -> /D4_P
- R8 pad 2: /Connectors/sheet5C922FED/DP0 -> /sheet5CBA03CA/DP4
- R9 pad 1: /Connectors/D3_P -> /D4_N
- R9 pad 2: /Connectors/sheet5C922FED/DP3 -> /sheet5CBA03CA/DM4
- U1 pad 1: /Connectors/SPI_MISO -> /BOARD_SENSE_1
- U1 pad 10: GND -> /BOARD_SENSE_3
- U1 pad 11: Net-(U1-Pad11) -> /JTAG_TDI
- U1 pad 12: Net-(U1-Pad12) -> /JTAG_TDO_3
- U1 pad 13: Net-(U1-Pad13) -> /BOARD_SENSE_4
- U1 pad 14: Net-(U1-Pad14) -> +3V3
- U1 pad 2: /Connectors/SPI_MOSI -> /JTAG_TDO
- U1 pad 3: /Connectors/SPI_SS -> /JTAG_TDO_1
- U1 pad 4: /Connectors/SPI_SCLK -> /BOARD_SENSE_2
- U1 pad 5: Net-(U1-Pad5) -> /JTAG_TDO_1
- U1 pad 6: Net-(U1-Pad6) -> /JTAG_TDO_2
- U1 pad 7: +3V3 -> GND
- U1 pad 8: +3V3 -> /JTAG_TDO_3
- U1 pad 9: +3V3 -> /JTAG_TDO_2
- U2 pad 2: Net-(U2-Pad2) -> Net-(R3-Pad1)
- U2 pad 3: Net-(R3-Pad1) -> /sheet5CBA03CA/DP0
- U2 pad 4: Net-(R3-Pad2) -> /sheet5CBA03CA/DM0
- U2 pad 6: Net-(U2-Pad6) -> /~SYSRESET
- U3 pad 1: /Connectors/sheet5C96EC1B/OSC1 -> Net-(U3-Pad1)
- U3 pad 2: /Connectors/sheet5C96EC1B/OSC0 -> Net-(U3-Pad2)
- U3 pad 3: Net-(C15-Pad2) -> Net-(R16-Pad1)
- U3 pad 4: GND -> Net-(R16-Pad2)
- U3 pad 5: Net-(R29-Pad1) -> GND
- U3 pad 6: /Connectors/sheet5C96EC1B/D- -> Net-(U3-Pad6)
- U3 pad 7: /Connectors/sheet5C96EC1B/D+ -> Net-(U3-Pad7)
- U3 pad 8: Net-(C16-Pad1) -> +3V3
- U4 pad 1: Net-(U4-Pad1) -> /sheet5CBA03CB/OSC1
- U4 pad 10: +3V3 -> GND
- U4 pad 11: Net-(U4-Pad11) -> GND
- U4 pad 12: Net-(U4-Pad12) -> +3V3
- U4 pad 13: /Connectors/sheet5C922FED/DM1 -> /JTAG_TCK
- U4 pad 14: /Connectors/sheet5C922FED/DP1 -> /JTAG_TDI
- U4 pad 15: Net-(U4-Pad15) -> /JTAG_TDO
- U4 pad 16: Net-(U4-Pad16) -> /JTAG_TMS
- U4 pad 17: /Connectors/sheet5C922FED/DM2 -> /~JTAG_TRST
- U4 pad 18: /Connectors/sheet5C922FED/DP2 -> /sheet5CBA03CB/ADBUS5
- U4 pad 2: Net-(R8-Pad1) -> /sheet5CBA03CB/OSC0
- U4 pad 21: /Connectors/sheet5C922FED/DM3 -> /sheet5CBA03CB/ACBUS0
- U4 pad 22: /Connectors/sheet5C922FED/DP3 -> GND
- U4 pad 23: Net-(U4-Pad23) -> GND
- U4 pad 24: Net-(U4-Pad24) -> +3V3
- U4 pad 26: /Connectors/sheet5C922FED/DM4 -> /sheet5CBA03CB/ACBUS2
- U4 pad 27: /Connectors/sheet5C922FED/DP4 -> /sheet5CBA03CB/ACBUS3
- U4 pad 3: /Connectors/sheet5C922FED/DP0 -> Net-(C15-Pad2)
- U4 pad 30: /Connectors/sheet5C922FED/DM5 -> /sheet5CBA03CB/ACBUS6
- U4 pad 31: /Connectors/sheet5C922FED/DP5 -> /sheet5CBA03CB/ACBUS7
- U4 pad 34: Net-(U4-Pad34) -> Net-(R18-Pad1)
- U4 pad 35: Net-(U4-Pad35) -> GND
- U4 pad 36: Net-(U4-Pad36) -> GND
- U4 pad 37: Net-(U4-Pad37) -> Net-(C13-Pad1)
- U4 pad 38: Net-(U4-Pad38) -> +1V8
- U4 pad 39: Net-(U4-Pad39) -> +3V3
- U4 pad 4: /Connectors/sheet5C922FED/DM0 -> GND
- U4 pad 40: Net-(U4-Pad40) -> +3V3
- U4 pad 41: Net-(U4-Pad41) -> GND
- U4 pad 42: Net-(U4-Pad42) -> GND
- U4 pad 43: GND -> Net-(R16-Pad1)
- U4 pad 44: Net-(C32-Pad2) -> Net-(U3-Pad2)
- U4 pad 45: Net-(C31-Pad2) -> Net-(U3-Pad1)
- U4 pad 47: +3V3 -> GND
- U4 pad 5: GND -> Net-(R19-Pad1)
- U4 pad 6: /Connectors/sheet5C922FED/~RESET -> /sheet5CBA03CB/D-
- U4 pad 7: Net-(U4-Pad7) -> /sheet5CBA03CB/D+
- U4 pad 8: +3V3 -> Net-(C16-Pad1)
- U4 pad 9: +3V3 -> GND
- Y1 pad 1: /TM4C129/OSC0 -> GND
- Y1 pad 2: GND -> Net-(C4-Pad2)
- Y1 pad 3: Net-(C4-Pad2) -> GND
- Y1 pad 4: GND -> Net-(C3-Pad2)
- Y2 pad 2: /Connectors/sheet5C96EC1B/OSC0_R -> /sheet5CBA03CB/OSC0_R
- Y2 pad 4: /Connectors/sheet5C96EC1B/OSC1 -> /sheet5CBA03CB/OSC1
Routing:
- net GND: track 250.6 -> 38.0 mm, vias 42 -> 5
- net /Connectors/JTAG_TDO_4: track 192.1 -> 0.00 mm, vias 1 -> 0
- net /JTAG_TCK: track 162.2 -> 0.00 mm, vias 1 -> 0
- net /JTAG_TMS: track 158.0 -> 0.03 mm, vias 3 -> 0
- net /Connectors/~JTAG_TRST: track 156.0 -> 0.00 mm, vias 1 -> 0
- net /Connectors/D4_P: track 153.1 -> 0.00 mm
- net /Connectors/D4_N: track 150.1 -> 0.00 mm
- net +3V3: track 126.9 -> 4.41 mm, vias 22 -> 2
- net /D3_P: track 0.00 -> 114.3 mm
- net /Connectors/D3_P: track 114.1 -> 0.00 mm
- net /Connectors/D3_N: track 111.0 -> 0.00 mm
- net /D3_N: track 0.00 -> 106.6 mm
- net /Connectors/D2_P: track 83.5 -> 0.00 mm
- net /Memory/EPIOS15: track 82.4 -> 0.00 mm, vias 3 -> 0
- net /Connectors/D2_N: track 80.4 -> 0.00 mm
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Other:
- board size 141.5 x 64.5 mm -> 120.7 x 64.1 mm
