File: ft232h.sch (KiCad schematic (older format))
At the start: 14 parts, among them U2 93LCxxB, U3 FT232H, Y2 Crystal

Commit message: usb hub and sdram selected.
Parts:
- removed Y2: Crystal, Crystal:Crystal_HC49-4H_Vertical, symbol Device:Crystal
- added R29: R_Small, symbol Device:R_Small
- added Y2: Crystal_GND24, Crystal:Crystal_SMD_3225-4Pin_3.2x2.5mm, symbol Device:Crystal_GND24
Connections:
- wire segments 104 -> 108
Other:
- moved on the sheet: C11, C12, C13, C14, C15, C16, L1, L2, R29, R3, R5, U2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

Commit message: schematics for expansion slots and memory
Parts:
- R29: footprint (none) -> Resistor_SMD:R_0603_1608Metric
Changed lines of the file:
@@
 $Descr A4 11693 8268
 encoding utf-8
-Sheet 3 5
+Sheet 5 10
 Title ""
 Date "2019-03-16"
@@
 F 0 "R4" V 4254 5300 50  0000 C CNN
 F 1 "R_Small" V 4345 5300 50  0000 C CNN
-F 2 "" H 4450 5300 50  0001 C CNN
+F 2 "Resistor_SMD:R_0603_1608Metric" H 4450 5300 50  0001 C CNN
 F 3 "~" H 4450 5300 50  0001 C CNN
 	1    4450 5300

Commit message: almost done with draft 1 of layout
Connections:
- net OSC1: now reaches C12.1, U3.1 (XCSI), Y2.4
- net OSC0: now reaches R29.1, U3.2 (XCSO)
- net OSC0_R: now reaches C14.1, R29.2, Y2.2
Changed lines of the file:
@@
 Wire Wire Line
 	4350 5100 4450 5100
+Text Label 4400 4900 0    50   ~ 0
+OSC1
+Text Label 4600 5300 0    50   ~ 0
+OSC0
+Text Label 3900 5300 0    50   ~ 0
+OSC0_R
 $EndSCHEMATC
