File: Exodus1000.sch (KiCad schematic (older format))
At the start: 5 parts, among them J1 USB_B_Mini, J3 Conn_01x02, U1 74LS125

Commit message: picking this back up. Removing old unused schematic sheets.
Parts:
- removed J1: USB_B_Mini, Connector_USB:USB_Mini-B_Lumberg_2486_01_Horizontal, symbol Connector:USB_B_Mini
- added C17, C18: C_Small, symbol Device:C_Small
- added J1: USB_B, symbol Connector:USB_B
- added J2: ARJ-169, symbol Exodus_Connectors:ARJ-169
Connections:
- net labels added: +5V
- net labels removed: D5_N, D5_P
- wire segments 96 -> 110
Changed lines of the file:
@@
 Wire Wire Line
 	1300 3500 1300 3600
-$Comp
-L Connector:USB_B_Mini J?
-U 1 1 5CBA03E0
-P 1300 3100
-AR Path="/5C8128A2/5CBA03E0" Ref="J?"  Part="1"
-AR Path="/5CBA03E0" Ref="J1"  Part="1"
-F 0 "J1" H 1355 3567 50  0000 C CNN
-F 1 "USB_B_Mini" H 1355 3476 50  0000 C CNN
-F 2 "Connector_USB:USB_Mini-B_Lumberg_2486_01_Horizontal" H 1450 3050 50  0001 C CNN
-F 3 "~" H 1450 3050 50  0001 C CNN
-	1    1300 3100
-	1    0    0    -1
-$EndComp
 Wire Wire Line
 	1200 3500 1300 3500
-Connection ~ 1300 3500
-$Sheet
-S 1700 4700 1150 1550
-U 5CBA03F2
-F0 "sheet5CBA03CA" 50
-F1 "usb_hub.sch" 50
-F2 "upstream_usb_p" I L 1700 4800 50
-F3 "upstream_usb_n" I L 1700 4900 50
-F4 "~RESET" I L 1700 5050 50
-F5 "D5_P" I R 2850 4950 50
-F6 "D5_N" I R 2850 5050 50
-F7 "D4_P" I R 2850 5250 50
-F8 "D4_N" I R 2850 5350 50
-F9 "D3_P" I R 2850 5500 50
-F10 "D3_N" I R 2850 5600 50
-F11 "D2_P" I R 2850 5750 50
-F12 "D2_N" I R 2850 5850 50
-F13 "D1_P" I R 2850 6000 50
-F14 "D1_N" I R 2850 6100 50
-$EndSheet
 $Sheet
 S 1850 2950 900  800
@@
 $EndSheet
 Wire Wire Line
-	2850 4950 3200 4950
-Wire Wire Line
-	2850 5050 3200 5050
-Wire Wire Line
 	2850 5250 3200 5250
 Wire Wire Line
@@
 Wire Wire Line
 	2850 6100 3200 6100
-Text Label 3200 4950 0    50   ~ 0
-D5_P
-Text Label 3200 5050 0    50   ~ 0
-D5_N
 Text Label 3200 5250 0    50   ~ 0
 D4_P
@@
 Text Label 7000 2250 2    50   ~ 0
 JTAG_TDO
-Wire Wire Line
-	1700 4800 1350 4800
-Wire Wire Line
-	1700 4900 1350 4900
-Text Label 1350 4800 0    50   ~ 0
+Text Label 1300 4800 0    50   ~ 0
 D0_P
-Text Label 1350 4900 0    50   ~ 0
+Text Label 1300 4900 0    50   ~ 0
 D0_N
-Wire Wire Line
-	1700 5050 1350 5050
-Text Label 1350 5050 2    50   ~ 0
+Text Label 1300 5050 0    50   ~ 0
 ~SYSRESET
 Text Label 3100 3150 0    50   ~ 0
@@
 Text Label 3100 3250 0    50   ~ 0
 JTAG_TDO
+$Comp
+L Connector:USB_B J1
+U 1 1 5D172A2C
+P 1300 3100
+F 0 "J1" H 1357 3567 50  0000 C CNN
+F 1 "USB_B" H 1357 3476 50  0000 C CNN
+F 2 "" H 1450 3050 50  0001 C CNN
+F 3 " ~" H 1450 3050 50  0001 C CNN
+	1    1300 3100
+	1    0    0    -1
+$EndComp
+Connection ~ 1300 3500
+$Comp
+L Exodus_Connectors:ARJ-169 J2
+U 2 1 5D1786DB
+P 1800 7100
+F 0 "J2" H 1800 7698 50  0000 C CNN
+F 1 "ARJ-169" H 1800 7607 50  0000 C CNN
+F 2 "" H 1950 7300 50  0001 C CNN
+F 3 "" H 1950 7300 50  0001 C CNN
+	2    1800 7100
+	1    0    0    -1
+$EndComp
+$Comp
+L Exodus_Connectors:ARJ-169 J2
+U 1 1 5D1824B2
+P 4200 6650
+F 0 "J2" H 4200 7475 50  0000 C CNN
+F 1 "ARJ-169" H 4200 7384 50  0000 C CNN
+F 2 "" H 4350 6850 50  0001 C CNN
+F 3 "" H 4350 6850 50  0001 C CNN
+	1    4200 6650
+	1    0    0    -1
+$EndComp
+Wire Wire Line
+	4600 6450 4800 6450
+Wire Wire Line
+	4600 6150 4800 6150
+$Comp
+L Device:C_Small C17
+U 1 1 5D1996E5
+P 4900 6150
+F 0 "C17" V 4671 6150 50  0000 C CNN
+F 1 "C_Small" V 4762 6150 50  0000 C CNN
+F 2 "" H 4900 6150 50  0001 C CNN
+F 3 "~" H 4900 6150 50  0001 C CNN
+	1    4900 6150
+	0    1    1    0
+$EndComp
+$Comp
+L Device:C_Small C18
+U 1 1 5D1999E2
+P 4900 6450
+F 0 "C18" V 4671 6450 50  0000 C CNN
+F 1 "C_Small" V 4762 6450 50  0000 C CNN
+F 2 "" H 4900 6450 50  0001 C CNN
+F 3 "~" H 4900 6450 50  0001 C CNN
+	1    4900 6450
+	0    1    1    0
+$EndComp
+$Comp
+L power:GND #PWR02
+U 1 1 5D199E52
+P 5150 6200
+F 0 "#PWR02" H 5150 5950 50  0001 C CNN
+F 1 "GND" H 5155 6027 50  0000 C CNN
+F 2 "" H 5150 6200 50  0001 C CNN
+F 3 "" H 5150 6200 50  0001 C CNN
+	1    5150 6200
+	1    0    0    -1
+$EndComp
+$Comp
+L power:GND #PWR03
+U 1 1 5D19A0F2
+P 5150 6500
+F 0 "#PWR03" H 5150 6250 50  0001 C CNN
+F 1 "GND" H 5155 6327 50  0000 C CNN
+F 2 "" H 5150 6500 50  0001 C CNN
+F 3 "" H 5150 6500 50  0001 C CNN
+	1    5150 6500
+	1    0    0    -1
+$EndComp
+Wire Wire Line
+	5000 6450 5150 6450
+Wire Wire Line
+	5150 6450 5150 6500
+Wire Wire Line
+	5000 6150 5150 6150
+Wire Wire Line
+	5150 6150 5150 6200
+Wire Wire Line
+	4600 6050 4800 6050
+Wire Wire Line
+	4600 6250 4800 6250
+Wire Wire Line
+	4600 6350 4800 6350
+Wire Wire Line
+	4600 6550 4800 6550
+Wire Wire Line
+	2100 7100 2300 7100
+Wire Wire Line
+	2100 7200 2300 7200
+Wire Wire Line
+	2100 7400 2300 7400
+Wire Wire Line
+	2300 7400 2300 7500
+$Comp
+L power:GND #PWR01
+U 1 1 5D1CD60E
+P 2300 7500
+F 0 "#PWR01" H 2300 7250 50  0001 C CNN
+F 1 "GND" H 2305 7327 50  0000 C CNN
+F 2 "" H 2300 7500 50  0001 C CNN
+F 3 "" H 2300 7500 50  0001 C CNN
+	1    2300 7500
+	1    0    0    -1
+$EndComp
+Text Label 2300 7200 0    50   ~ 0
+D4_P
+Text Label 2300 7100 0    50   ~ 0
+D4_N
+$Sheet
+S 1700 4700 1150 1550
+U 5CBA03F2
+F0 "sheet5CBA03CA" 50
+F1 "usb_hub.sch" 50
+F2 "upstream_usb_p" I L 1700 4800 50
+F3 "upstream_usb_n" I L 1700 4900 50
+F4 "~RESET" I L 1700 5050 50
+F5 "D3_P" I R 2850 5500 50
+F6 "D3_N" I R 2850 5600 50
+F7 "D1_P" I R 2850 6000 50
+F8 "D1_N" I R 2850 6100 50
+F9 "D4_N" I R 2850 5350 50
+F10 "D4_P" I R 2850 5250 50
+F11 "D2_P" I R 2850 5750 50
+F12 "D2_N" I R 2850 5850 50
+$EndSheet
+Wire Wire Line
+	2100 6900 2300 6900
+Wire Wire Line
+	2300 6900 2300 6800
+$Comp
+L power:+5V #PWR?
+U 1 1 5D20275C
+P 2300 6800
+F 0 "#PWR?" H 2300 6650 50  0001 C CNN
+F 1 "+5V" H 2315 6973 50  0000 C CNN
+F 2 "" H 2300 6800 50  0001 C CNN
+F 3 "" H 2300 6800 50  0001 C CNN
+	1    2300 6800
+	1    0    0    -1
+$EndComp
+Wire Wire Line
+	1300 5050 1700 5050
+Wire Wire Line
+	1300 4900 1700 4900
+Wire Wire Line
+	1300 4800 1700 4800
 $EndSCHEMATC
