File: expansion_slot.sch (KiCad schematic (older format))
At the start: 1 part, among them M1 ET60S-02-24-02-X-VP-GP

Commit message: almost done with draft 1 of layout
Parts:
- added R31: R_Small, Resistor_SMD:R_0603_1608Metric, symbol Device:R_Small
Connections:
- net BOARD_SENSE: now also R31.1
- net GND: now also R31.2
- net USB_N: now also M1.1; no longer M1.2
- net USB_P: now also M1.2; no longer M1.1
- net ~INHIBIT: now also M1.16; no longer M1.9
Changed lines of the file:
@@
 $Descr A4 11693 8268
 encoding utf-8
-Sheet 9 10
+Sheet 8 10
 Title ""
 Date ""
@@
 AR Path="/5C8128A2/5C97B51C/5C9582A1" Ref="M3"  Part="1"
 AR Path="/5C8128A2/5C97B7CC/5C9582A1" Ref="M4"  Part="1"
-F 0 "M4" H 6828 1042 45  0000 L CNN
+F 0 "M2" H 6828 1042 45  0000 L CNN
 F 1 "ET60S-02-24-02-X-VP-GP" H 6828 958 45  0000 L CNN
 F 2 "Exodus_Connectors:ET60S-02-24-02-X-VP-GP" H 6330 2300 20  0001 C CNN
@@
 AR Path="/5C8128A2/5C97B51C/5C9582A8" Ref="M3"  Part="2"
 AR Path="/5C8128A2/5C97B7CC/5C9582A8" Ref="M4"  Part="2"
-F 0 "M4" H 4550 2754 45  0000 C CNN
+F 0 "M2" H 4550 2754 45  0000 C CNN
 F 1 "ET60S-02-24-02-X-VP-GP" H 4550 2670 45  0000 C CNN
 F 2 "Exodus_Connectors:ET60S-02-24-02-X-VP-GP" H 4130 2650 20  0001 C CNN
@@
 Wire Wire Line
 	6300 2650 6100 2650
+Text HLabel 6100 2250 0    50   Input ~ 0
+USB_P
 Text HLabel 6100 2150 0    50   Input ~ 0
-USB_P
-Text HLabel 6100 2250 0    50   Input ~ 0
 USB_N
 Text HLabel 6100 2650 0    50   Input ~ 0
@@
 	6300 2850 6100 2850
 Wire Wire Line
-	6300 2950 6100 2950
+	6300 3650 6100 3650
 Text HLabel 6100 2850 0    50   Input ~ 0
 ~ENABLE
-Text HLabel 6100 2950 0    50   Input ~ 0
+Text HLabel 6100 3650 0    50   Input ~ 0
 ~INHIBIT
 Wire Wire Line
@@
 Text HLabel 6100 3150 0    50   Input ~ 0
 ~SYSRESET
+Text Label 2850 2650 0    50   ~ 0
+BOARD_SENSE
+$Comp
+L Device:R_Small R?
+U 1 1 5CD70420
+P 2600 2850
+AR Path="/5C8128A2/5CD70420" Ref="R?"  Part="1"
+AR Path="/5C8128A2/5C947A1C/5CD70420" Ref="R31"  Part="1"
+AR Path="/5C8128A2/5C97B26C/5CD70420" Ref="R32"  Part="1"
+AR Path="/5C8128A2/5C97B51C/5CD70420" Ref="R33"  Part="1"
+AR Path="/5C8128A2/5C97B7CC/5CD70420" Ref="R35"  Part="1"
+F 0 "R32" H 2659 2896 50  0000 L CNN
+F 1 "R_Small" H 2659 2805 50  0000 L CNN
+F 2 "Resistor_SMD:R_0603_1608Metric" H 2600 2850 50  0001 C CNN
+F 3 "~" H 2600 2850 50  0001 C CNN
+	1    2600 2850
+	1    0    0    -1
+$EndComp
+Wire Wire Line
+	2600 2950 2600 3050
+$Comp
+L power:GND #PWR?
+U 1 1 5CD70428
+P 2600 3050
+AR Path="/5C8128A2/5CD70428" Ref="#PWR?"  Part="1"
+AR Path="/5C8128A2/5C947A1C/5CD70428" Ref="#PWR0185"  Part="1"
+AR Path="/5C8128A2/5C97B26C/5CD70428" Ref="#PWR0186"  Part="1"
+AR Path="/5C8128A2/5C97B51C/5CD70428" Ref="#PWR0187"  Part="1"
+AR Path="/5C8128A2/5C97B7CC/5CD70428" Ref="#PWR0192"  Part="1"
+F 0 "#PWR0192" H 2600 2800 50  0001 C CNN
+F 1 "GND" H 2605 2877 50  0000 C CNN
+F 2 "" H 2600 3050 50  0001 C CNN
+F 3 "" H 2600 3050 50  0001 C CNN
+	1    2600 3050
+	1    0    0    -1
+$EndComp
+Wire Wire Line
+	2600 2750 2600 2650
+Wire Wire Line
+	2600 2650 2850 2650
 $EndSCHEMATC

Commit message: layout done sans connector. It's pretty big. Likely going to need to tear some of this up.
Changed lines of the file:
@@
 AR Path="/5C8128A2/5C97B51C/5C9582A1" Ref="M3"  Part="1"
 AR Path="/5C8128A2/5C97B7CC/5C9582A1" Ref="M4"  Part="1"
-F 0 "M2" H 6828 1042 45  0000 L CNN
+F 0 "M4" H 6828 1042 45  0000 L CNN
 F 1 "ET60S-02-24-02-X-VP-GP" H 6828 958 45  0000 L CNN
 F 2 "Exodus_Connectors:ET60S-02-24-02-X-VP-GP" H 6330 2300 20  0001 C CNN
@@
 AR Path="/5C8128A2/5C97B51C/5C9582A8" Ref="M3"  Part="2"
 AR Path="/5C8128A2/5C97B7CC/5C9582A8" Ref="M4"  Part="2"
-F 0 "M2" H 4550 2754 45  0000 C CNN
+F 0 "M4" H 4550 2754 45  0000 C CNN
 F 1 "ET60S-02-24-02-X-VP-GP" H 4550 2670 45  0000 C CNN
 F 2 "Exodus_Connectors:ET60S-02-24-02-X-VP-GP" H 4130 2650 20  0001 C CNN
@@
 AR Path="/5C8128A2/5C97B51C/5CD70420" Ref="R33"  Part="1"
 AR Path="/5C8128A2/5C97B7CC/5CD70420" Ref="R35"  Part="1"
-F 0 "R32" H 2659 2896 50  0000 L CNN
+F 0 "R35" H 2659 2896 50  0000 L CNN
 F 1 "R_Small" H 2659 2805 50  0000 L CNN
 F 2 "Resistor_SMD:R_0603_1608Metric" H 2600 2850 50  0001 C CNN

Commit message: this is just a mess. but I think the schematic is basically right still.
Parts:
- removed M1: ET60S-02-24-02-X-VP-GP, Exodus_Connectors:ET60S-02-24-02-X-VP-GP, symbol ET60S-02-24-02-X-VP-GP:ET60S-02-24-02-X-VP-GP
- added 3: ET60S-02-24-02-X-VP-GP, Exodus_Connectors:ET60S-02-24-02-X-VP-GP, symbol Exodus_Connectors:ET60S-02-24-02-X-VP-GP
Connections:
- net +3V3: now also 3.P4-1 (25), 3.P4-2 (26), 3.P4-3 (27), 3.P4-4 (28), 3.P4-5 (29), 3.P4-6 (30), 3.P4-7 (31), 3.P4-8 (32)
- net +5V: now also 3.P3-1 (17), 3.P3-2 (18), 3.P3-3 (19), 3.P3-4 (20), 3.P3-5 (21), 3.P3-6 (22), 3.P3-7 (23), 3.P3-8 (24)
- net +BATT: now also 3.P2-1 (9), 3.P2-2 (10), 3.P2-3 (11), 3.P2-4 (12), 3.P2-5 (13), 3.P2-6 (14), 3.P2-7 (15), 3.P2-8 (16)
- net BOARD_SENSE: now also 3.10
- net GND: now also 3.P1-1 (1), 3.P1-2 (2), 3.P1-3 (3), 3.P1-4 (4), 3.P1-5 (5), 3.P1-6 (6), 3.P1-7 (7), 3.P1-8 (8)
- net JTAG_TCK: now also 3.6
- net JTAG_TDI: now also 3.4
- net JTAG_TDO: now also 3.5
- net JTAG_TMS: now also 3.3
- net USB_N: now also 3.1
- net USB_P: now also 3.2
- net ~ENABLE: now also 3.8
- net ~INHIBIT: now also 3.16
- net ~JTAG_TRST: now also 3.7
- net ~SYSRESET: now also 3.11

Commit message: picking this back up. Removing old unused schematic sheets.
Parts:
- renumbered 3 to 31
Changed lines of the file:
@@
 $Descr A4 11693 8268
 encoding utf-8
-Sheet 7 7
+Sheet 6 7
 Title ""
 Date ""
@@
 	2600 2650 2850 2650
 $Comp
-L Exodus_Connectors:ET60S-02-24-02-X-VP-GP 3
+L Exodus_Connectors:ET60S-02-24-02-X-VP-GP 31
 U 1 1 5CD0546A
 P 6300 2150
-AR Path="/5CBA042A/5CD0546A" Ref="3"  Part="1"
-AR Path="/5CBA0410/5CD0546A" Ref="1"  Part="1"
-AR Path="/5CBA041D/5CD0546A" Ref="2"  Part="1"
-AR Path="/5CBA0437/5CD0546A" Ref="4"  Part="1"
-F 0 "4" H 6828 1040 42  0000 L CNN
+AR Path="/5CBA042A/5CD0546A" Ref="31"  Part="1"
+AR Path="/5CBA0410/5CD0546A" Ref="11"  Part="1"
+AR Path="/5CBA041D/5CD0546A" Ref="21"  Part="1"
+AR Path="/5CBA0437/5CD0546A" Ref="41"  Part="1"
+F 0 "41" H 6828 1040 42  0000 L CNN
 F 1 "ET60S-02-24-02-X-VP-GP" H 6828 961 42  0000 L CNN
 F 2 "Exodus_Connectors:ET60S-02-24-02-X-VP-GP" H 6300 2150 50  0001 C CNN
@@
 	4050 3700 4050 3800
 $Comp
-L Exodus_Connectors:ET60S-02-24-02-X-VP-GP 3
+L Exodus_Connectors:ET60S-02-24-02-X-VP-GP 31
 U 2 1 5CD08AE4
 P 4100 2500
-AR Path="/5CBA042A/5CD08AE4" Ref="3"  Part="2"
-AR Path="/5CBA0410/5CD08AE4" Ref="1"  Part="2"
-AR Path="/5CBA041D/5CD08AE4" Ref="2"  Part="2"
-AR Path="/5CBA0437/5CD08AE4" Ref="4"  Part="2"
-F 0 "4" H 4550 2747 42  0000 C CNN
+AR Path="/5CBA042A/5CD08AE4" Ref="31"  Part="2"
+AR Path="/5CBA0410/5CD08AE4" Ref="11"  Part="2"
+AR Path="/5CBA041D/5CD08AE4" Ref="21"  Part="2"
+AR Path="/5CBA0437/5CD08AE4" Ref="41"  Part="2"
+F 0 "41" H 4550 2747 42  0000 C CNN
 F 1 "ET60S-02-24-02-X-VP-GP" H 4550 2668 42  0000 C CNN
 F 2 "Exodus_Connectors:ET60S-02-24-02-X-VP-GP" H 4100 2500 50  0001 C CNN
